Commit message: demo improvements

File: resources/robots/stretch.urdf (robot description, URDF)
Before this commit: robot stretch, 46 links, 45 joints
Links:
- link base_imu: mass 0.000901473198307758 -> 0.00092
- link base_link: mass 1.1912 -> None
- link laser: mass 0.0749979022894495 -> 0.216007
- link link_arm_l0: mass 0.085003260946398 -> 0.427734
- link link_arm_l1: mass 0.051382 -> 0.113658
- link link_arm_l2: mass 0.0571386353275368 -> 0.130565
- link link_arm_l3: mass 0.0628927381893134 -> 0.146817
- link link_arm_l4: mass 0.068095 -> 0.235626
- link link_aruco_inner_wrist: mass 0.0 -> 0
- link link_aruco_left_base: mass 3.59999999990368e-06 -> 3.59999999990368E-06
- link link_aruco_right_base: mass 3.59999999990368e-06 -> 3.59999999990368E-06
- link link_aruco_shoulder: mass 0.0 -> 0
- link link_aruco_top_wrist: mass 0.0 -> 0
- link link_head: mass 0.133027236718691 -> 0.681871
- link link_head_pan: mass 0.0273764496535409 -> 0.062462
- link link_head_tilt: mass 0.090217113313934 -> 0.283548
- link link_left_wheel: mass 0.0042721 -> 0.20773
- link link_lift: mass 0.27218 -> 1.987167
- link link_mast: mass 1.8285 -> 1.764017
- link link_right_wheel: mass 0.0042721 -> 0.20773
- link link_wrist_yaw: mass 0.0404746907425003 -> 0.054422
- link respeaker_base: mass 0.015643 -> 0.025175
Joints:
- joint camera_accel_joint: origin xyz=-0.01174 -0.00552 0.0051 rpy=0.0 0.0 0.0 -> xyz=-0.01174 -0.00552 0.0051 rpy=0 0 0
- joint camera_accel_optical_joint: origin xyz=0.0 0.0 0.0 rpy=-1.5707963267948966 0.0 -1.5707963267948966 -> xyz=0 0 0 rpy=-1.5707963267948966 0 -1.5707963267948966
- joint camera_color_joint: origin xyz=0.0 0.015 0.0 rpy=0.0 0.0 0.0 -> xyz=0 0.015 0 rpy=0 0 0
- joint camera_color_optical_joint: origin xyz=0.0 0.0 0.0 rpy=-1.5707963267948966 0.0 -1.5707963267948966 -> xyz=0 0 0 rpy=-1.5707963267948966 0 -1.5707963267948966
- joint camera_depth_joint: origin xyz=0.0 0.0 0.0 rpy=0.0 0.0 0.0 -> xyz=0 0 0 rpy=0 0 0
- joint camera_depth_optical_joint: origin xyz=0.0 0.0 0.0 rpy=-1.5707963267948966 0.0 -1.5707963267948966 -> xyz=0 0 0 rpy=-1.5707963267948966 0 -1.5707963267948966
- joint camera_gyro_joint: origin xyz=-0.01174 -0.00552 0.0051 rpy=0.0 0.0 0.0 -> xyz=-0.01174 -0.00552 0.0051 rpy=0 0 0
- joint camera_gyro_optical_joint: origin xyz=0.0 0.0 0.0 rpy=-1.5707963267948966 0.0 -1.5707963267948966 -> xyz=0 0 0 rpy=-1.5707963267948966 0 -1.5707963267948966
- joint camera_infra1_joint: origin xyz=0.0 0.0 0.0 rpy=0.0 0.0 0.0 -> xyz=0 0.0 0 rpy=0 0 0
- joint camera_infra1_optical_joint: origin xyz=0.0 0.0 0.0 rpy=-1.5707963267948966 0.0 -1.5707963267948966 -> xyz=0 0 0 rpy=-1.5707963267948966 0 -1.5707963267948966
- joint camera_infra2_joint: origin xyz=0.0 -0.05 0.0 rpy=0.0 0.0 0.0 -> xyz=0 -0.05 0 rpy=0 0 0
- joint camera_infra2_optical_joint: origin xyz=0.0 0.0 0.0 rpy=-1.5707963267948966 0.0 -1.5707963267948966 -> xyz=0 0 0 rpy=-1.5707963267948966 0 -1.5707963267948966
- joint camera_joint: origin xyz=0.025518771292122495 -0.010053319210363395 0.01844042865675001 rpy=0.0012927647205987253 -0.049412987457166935 0.0012120493497760406 -> xyz=0.03 -0.0122 0.0182 rpy=0.0 0.0 0.0
- joint camera_link_joint: origin xyz=0.010600000000000002 0.0175 0.0125 rpy=0.0 0.0 0.0 -> xyz=0.010600000000000002 0.0175 0.0125 rpy=0 0 0
- joint caster_joint: axis 0.0 0.0 1.0 -> 0 0 1; origin xyz=-0.245 0.0 0.032 rpy=-1.5707963267948966 0.0 0.0 -> xyz=-0.245 0.0 0.032 rpy=-1.5707963267948966 0 0
- joint joint_arm_l0: axis 0.0 0.0 1.0 -> 0 0 1; limit lower=0.0 upper=0.13 effort=100.0 velocity=1.0 -> lower=0.0 upper=0.13 effort=100 velocity=1.0; origin xyz=0.0 0.0 -0.0137499999991968 rpy=7.63746778746202e-30 -3.80121128864402e-15 2.62707547767438e-15 -> xyz=0 0 -0.0137499999991968 rpy=7.63746778746202E-30 -3.80121128864402E-15 2.62707547767438E-15
- joint joint_arm_l1: axis 0.0 0.0 1.0 -> 0 0 1; limit lower=0.0 upper=0.13 effort=100.0 velocity=1.0 -> lower=0.0 upper=0.13 effort=100 velocity=1.0; origin xyz=0.0 0.0 0.0129999999999981 rpy=-7.63746778746202e-30 -7.88860905221012e-31 1.11022302462516e-16 -> xyz=0 0 0.0129999999999981 rpy=-7.63746778746202E-30 -7.88860905221012E-31 1.11022302462516E-16
- joint joint_arm_l2: axis 0.0 0.0 1.0 -> 0 0 1; limit lower=0.0 upper=0.13 effort=100.0 velocity=1.0 -> lower=0.0 upper=0.13 effort=100 velocity=1.0; origin xyz=0.0 0.0 0.013 rpy=0.0 1.57655765344625e-30 -1.66533453693773e-16 -> xyz=0 0 0.013 rpy=0 1.57655765344625E-30 -1.66533453693773E-16
- joint joint_arm_l3: axis 0.0 0.0 1.0 -> 0 0 1; limit lower=0.0 upper=0.13 effort=100.0 velocity=1.0 -> lower=0.0 upper=0.13 effort=100 velocity=1.0; origin xyz=0.0 0.0 0.013 rpy=7.68831233799385e-30 2.36716479416092e-30 2.29652732251143e-17 -> xyz=0 0 0.013 rpy=7.68831233799385E-30 2.36716479416092E-30 2.29652732251143E-17
- joint joint_arm_l4: axis 0.0 0.0 0.0 -> 0 0 0; origin xyz=-0.24976370113857183 -0.0038350045015007497 -0.0018596582600665607 rpy=1.576330969843221 0.0029295139899749856 -1.5981368109983811 -> xyz=-0.2547 0 0 rpy=1.5708 2.4721E-15 -1.5708
- joint joint_aruco_inner_wrist: axis 0.0 0.0 0.0 -> 0 0 0; origin xyz=0.0472499999999947 -0.0119000000000034 -0.0272499999991938 rpy=3.14159265358979 4.23377442363088e-14 3.14159265358979 -> xyz=0.0472499999999947 -0.0119000000000034 -0.0272499999991938 rpy=3.14159265358979 4.23377442363088E-14 3.14159265358979
- joint joint_aruco_left_base: axis 0.0 0.0 0.0 -> 0 0 0; origin xyz=-0.00500000000000014 0.1304972 0.1597482 rpy=0.0 0.0 -1.5707963267949 -> xyz=-0.00500000000000014 0.1304972 0.1597482 rpy=0 0 -1.5707963267949
- joint joint_aruco_right_base: axis 0.0 0.0 0.0 -> 0 0 0; origin xyz=-0.0015028 -0.1304972 0.1597482 rpy=0.0 0.0 -1.5707963267949 -> xyz=-0.0015028 -0.1304972 0.1597482 rpy=0 0 -1.5707963267949
- joint joint_aruco_shoulder: axis 0.0 0.0 0.0 -> 0 0 0; origin xyz=-0.0133768876375287 0.0558540528812078 0.0861368272417975 rpy=-1.53998860117704e-29 3.55962409571165e-15 0.0 -> xyz=-0.0133768876375287 0.0558540528812078 0.0861368272417975 rpy=-1.53998860117704E-29 3.55962409571165E-15 0.0
- joint joint_aruco_top_wrist: axis 0.0 0.0 0.0 -> 0 0 0; origin xyz=0.0472500000000019 0.0292850000000015 0.0 rpy=1.5707963267949 -8.03728587323464e-15 3.14159265358979 -> xyz=0.0472500000000019 0.0292850000000015 0 rpy=1.5707963267949 -8.03728587323464E-15 3.14159265358979
- joint joint_base_imu: axis 0.0 0.0 0.0 -> 0 0 0; origin xyz=-0.12838 0.0031592 0.1474 rpy=-3.1416 0.0 -1.5708 -> xyz=-0.12838 0.0031592 0.1474 rpy=-3.1416 0 -1.5708
- joint joint_grasp_center: origin xyz=0.0 0.0 0.23 rpy=-1.5707963267949 -1.5707963267949 0.0 -> xyz=0 0 0.23 rpy=-1.5707963267949 -1.5707963267949 0
- joint joint_gripper_finger_left: axis 0.0 0.0 -1.0 -> 0 0 -1; limit lower=-0.6 upper=0.6 effort=100.0 velocity=1.0 -> lower=-0.6 upper=0.6 effort=100 velocity=1.0; origin xyz=0.018599 0.003 0.033689 rpy=1.5708 -1.5708 0.0 -> xyz=0.018599 0.003 0.033689 rpy=1.5708 -1.5708 0
- joint joint_gripper_finger_right: axis 0.0 0.0 1.0 -> 0 0 1; limit lower=-0.6 upper=0.6 effort=100.0 velocity=1.0 -> lower=-0.6 upper=0.6 effort=100 velocity=1.0; origin xyz=-0.018599 0.003 0.033689 rpy=1.5708 1.5708 0.0 -> xyz=-0.018599 0.003 0.033689 rpy=1.5708 1.5708 0
- joint joint_gripper_fingertip_left: axis 0.0 0.0 0.0 -> 0 0 0; origin xyz=0.190596948563868 -0.015 0.0 rpy=1.57079632679496 4.51275387511463e-14 2.60113659715756 -> xyz=0.190596948563868 -0.015 0 rpy=1.57079632679496 4.51275387511463E-14 2.60113659715756
- joint joint_gripper_fingertip_right: axis 0.0 0.0 0.0 -> 0 0 0; origin xyz=-0.190596948563868 -0.015 0.0 rpy=-1.57079632679483 -3.43320051448326e-14 0.540456056432235 -> xyz=-0.190596948563868 -0.015 0 rpy=-1.57079632679483 -3.43320051448326E-14 0.540456056432235
- joint joint_head: axis 0.0 0.0 0.0 -> 0 0 0; origin xyz=0.0 1.33 0.0 rpy=1.5707963267949 -1.5707963267949 3.1416 -> xyz=0 1.33 0 rpy=1.5707963267949 -1.5707963267949 3.1416
- joint joint_head_pan: axis 0.0 0.0 1.0 -> 0 0 1; limit lower=-3.9 upper=1.5 effort=100.0 velocity=1.0 -> lower=-3.9 upper=1.5 effort=100 velocity=1.0; origin xyz=0.13034914529901984 0.07720989078406804 -0.009943382462533366 rpy=-0.006540305695066827 0.005914541231504256 1.5775160215215478 -> xyz=0.135 0.0731000000000001 -0.00319621125547975 rpy=0 0 1.5707963267949
- joint joint_head_tilt: axis 0.0 0.0 1.0 -> 0 0 1; limit lower=-1.53 upper=0.79 effort=100.0 velocity=1.0 -> lower=-1.53 upper=0.79 effort=100 velocity=1.0; origin xyz=-0.0022608566011374713 0.0307623849887207 -0.06164750121121569 rpy=1.6137456215249617 0.0264597080068929 -0.025133837247576386 -> xyz=-0.00130000001785262 0.0277624999926072 -0.0533107920897029 rpy=1.5707963267949 3.36459255518345E-15 -8.42914893687103E-17
- joint joint_laser: axis 0.0 0.0 0.0 -> 0 0 0; origin xyz=0.004 0.0 0.1664 rpy=0.0 0.0 3.1416 -> xyz=0.004 0 0.1664 rpy=0 0 3.1416
- joint joint_left_wheel: axis 0.0 0.0 1.0 -> 0 0 1; origin xyz=0.0 0.17035 0.0508 rpy=-1.5708 2.6317e-16 -8.2057e-19 -> xyz=0 0.17035 0.0508 rpy=-1.5708 2.6317E-16 -8.2057E-19
- joint joint_lift: axis 0.0 0.0 1.0 -> 0 0 1; limit lower=0.0 upper=1.1 effort=100.0 velocity=1.0 -> lower=0.0 upper=1.1 effort=100 velocity=1.0; origin xyz=-0.037385 0.1666 0.0 rpy=-1.5708 1.5708 0.0 -> xyz=-0.037385 0.1666 0 rpy=-1.5708 1.5708 0
- joint joint_mast: axis 0.0 0.0 0.0 -> 0 0 0; origin xyz=-0.06647627777956927 0.13686815294798188 0.02476215878246698 rpy=1.5835422401336123 0.009918315177623871 -0.001695598806231402 -> xyz=-0.067 0.135 0.0284 rpy=1.5708 0 4.8006E-17
- joint joint_respeaker: axis 0.0 0.0 0.0 -> 0 0 0; origin xyz=0.0 1.37236408874452 0.00303065898329655 rpy=-1.5707963267949 -0.698131700797725 4.93295812652799e-16 -> xyz=0 1.37236408874452 0.00303065898329655 rpy=-1.5707963267949 -0.698131700797725 4.93295812652799E-16
- joint joint_right_wheel: axis 0.0 0.0 1.0 -> 0 0 1; origin xyz=0.0 -0.17035 0.0508 rpy=-1.5708 1.2717e-16 4.8006e-17 -> xyz=0 -0.17035 0.0508 rpy=-1.5708 1.2717E-16 4.8006E-17
- joint joint_straight_gripper: axis 0.0 0.0 0.0 -> 0 0 0; origin xyz=0.0 0.0 0.0155 rpy=3.54987407349455e-30 3.24021254484265e-20 -3.14159265358979 -> xyz=0 0 0.0155 rpy=3.54987407349455E-30 3.24021254484265E-20 -3.14159265358979
- joint joint_wrist_pitch: axis 0.0 0.0 -1.0 -> 0 0 -1; limit lower=-1.57 upper=0.56 effort=100.0 velocity=1.0 -> lower=-1.57 upper=0.56 effort=100 velocity=1.0; origin xyz=0.0 -0.0195500000000002 -0.0247499999999984 rpy=1.5707963267949 -8.12895570882604e-15 -3.14159265358979 -> xyz=0 -0.0195500000000002 -0.0247499999999984 rpy=1.5707963267949 -8.12895570882604E-15 -3.14159265358979
- joint joint_wrist_roll: axis 0.0 0.0 1.0 -> 0 0 1; limit lower=-3.14 upper=3.14 effort=100.0 velocity=1.0 -> lower=-3.14 upper=3.14 effort=100 velocity=1.0; origin xyz=-0.0188587444076125 -0.0239999999998942 0.01955 rpy=3.14159265358979 1.5707963267949 0.0 -> xyz=-0.0188587444076125 -0.0239999999998942 0.01955 rpy=3.14159265358979 1.5707963267949 0
- joint joint_wrist_yaw: axis 0.0 0.0 -1.0 -> 0 0 -1; limit lower=-1.75 upper=4.0 effort=100.0 velocity=1.0 -> lower=-1.75 upper=4.0 effort=100 velocity=1.0; origin xyz=0.0830000000000654 -0.0307500000000129 0.0 rpy=1.5708 4.2595e-14 2.6415e-15 -> xyz=0.0830000000000654 -0.0307500000000129 0 rpy=1.5708 4.2595E-14 2.6415E-15
- joint joint_wrist_yaw_bottom: axis 0.0 0.0 0.0 -> 0 0 0; origin xyz=0.0 0.0 0.0 rpy=-3.14159265358979 1.13367999021379e-14 1.57079632679489 -> xyz=0 0 0 rpy=-3.14159265358979 1.13367999021379E-14 1.57079632679489
